Commit message: Modificació README

File: ddsr_description/urdf/ddsr_partial.xacro (robot description, xacro)
@@ -85,4 +85,5 @@
 	</inertial>
 </link>
+<!-- ~~~~~~~~~~~~~~~~~~~~~~~ DRIVE WHEELS ~~~~~~~~~~~~~~~~~~~~~~~~~~~~~~~~~~~~~~~~ -->
 <joint name="platform_2_left_wheel" type="continuous" >
 	<parent link="platform"/>
@@ -235,3 +236,56 @@
 	</inertial>
 </link>
+<joint name="caster_hinge_2_2_caster_wheel" type="continuous" >
+	<parent link="caster_hinge_2"/>
+	<child link="caster_wheel"/>
+	<origin xyz="0 0 ${-0.04*0.707*0.5}" rpy="-${0.5*pi} 0 0"/>
+	<axis xyz="0 0 1"/>
+	<limit effort="99999" velocity="${20*pi}"/>
+	<dynamics friction="0.25" damping="0.05"/>
+</joint>
+<link name="caster_wheel">
+	<visual>
+		<origin xyz="0 0 0" rpy="0 0 0"/>
+		<geometry>
+			<cylinder length="${0.5*wheel_width}" radius="${floor_clearance-0.02-0.04*0.707}"/>
+		</geometry>
+		<material name="ddsr/grey" />
+	</visual>
+	<collision>
+		<origin xyz="0 0 0" rpy="0 0 0"/>
+		<geometry>
+			<cylinder length="${0.5*wheel_width}" radius="${floor_clearance-0.02-0.04*0.707}"/>
+		</geometry>
+	</collision>
+	<inertial>
+		<mass value="${wheel_mass*0.5}" />
+		<origin xyz="0 0 0" rpy="0 0 0"/>
+		<inertia ixx="${0.083*wheel_mass*0.5*(3*wheel_radius*wheel_radius+wheel_width*wheel_width)}"
+			ixy="0.0"
+			ixz="0.0"
+			iyy="${0.083*wheel_mass*0.5*(3*wheel_radius*wheel_radius+wheel_width*wheel_width)}"
+			iyz="0.0"
+			izz="${0.5*wheel_mass*0.5*wheel_radius*wheel_radius}" />
+	</inertial>
+</link>
+<!--  caster steering free transmission -->
+<transmission name="platform_2_caster_hinge_1_transmission">
+	<type>transmission_interface/SimpleTransmission</type>
+	<joint name="platform_2_caster_hinge_1">
+		<hardwareInterface>hardware_interface/EffortJointInterface</hardwareInterface>
+	</joint>
+	<actuator name="platform_2_caster_hinge_1_steering">
+		<mechanicalReduction>1</mechanicalReduction>
+	</actuator>
+</transmission>
+<!-- caster drive free transmission -->
+<transmission name="caster_hinge_2_2_caster_wheel_transmission">
+	<type>transmission_interface/SimpleTransmission</type>
+	<joint name="caster_hinge_2_2_caster_wheel">
+		<hardwareInterface>hardware_interface/EffortJointInterface</hardwareInterface>
+	</joint>
+	<actuator name="caster_hinge_2_2_caster_driving">
+		<mechanicalReduction>1</mechanicalReduction>
+	</actuator>
+</transmission>
 </robot>
